Commit message: Overtake Node running, but not working

File: urdf/edison0.urdf (robot description, URDF)
Before this commit: robot Edison, 9 links, 8 joints
Joints:
- joint joint_wheel_left: axis (none) -> 0 1 0
- joint joint_wheel_right: axis (none) -> 0 1 0

File: urdf/edison1.urdf (robot description, URDF)
Before this commit: robot Edison, 9 links, 8 joints
Joints:
- joint joint_wheel_left: axis (none) -> 0 1 0
- joint joint_wheel_right: axis (none) -> 0 1 0
